File: 12VBuckBoost.kicad_pcb (KiCad board)
At the start: 2 copper layers, 24 parts, among them J1 Conn_01x02, J2 Conn_01x01, J3 QWIIC, J4 Conn_01x02, U1 TPS55289RYQR

Commit message: Init
Parts:
- removed C10: 22uF, Capacitor_SMD:C_1210_3225Metric_Pad1.33x2.70mm_HandSolder
- removed C7, C8, C9: 22uF X7R, Capacitor_SMD:C_1210_3225Metric_Pad1.33x2.70mm_HandSolder
- removed J2: Conn_01x01, Connector_PinHeader_2.54mm:PinHeader_1x01_P2.54mm_Vertical
- removed J3: QWIIC, Connector_JST:JST_PH_S4B-PH-K_1x04_P2.00mm_Horizontal
- removed J4: Conn_01x02, Connector_PinHeader_2.54mm:PinHeader_1x02_P2.54mm_Vertical
- removed R6: 4.7k, Resistor_SMD:R_1210_3225Metric_Pad1.30x2.65mm_HandSolder
- added C14: 330uF, ZKU Capacitors:CAP_ZKU_F_PAN, F.Cu at (125.2, 73.8)
- added R4: 10m, Resistor_SMD:R_0805_2012Metric_Pad1.20x1.40mm_HandSolder, F.Cu at (141.0, 74.1)
- C1, C2: value 22uF -> 0.1uF; footprint Capacitor_SMD:C_1210_3225Metric_Pad1.33x2.70mm_HandSolder -> Capacitor_SMD:C_0805_2012Metric_Pad1.18x1.45mm_HandSolder
- C13: value 22uF X7R -> 330uF; footprint Capacitor_SMD:C_1210_3225Metric_Pad1.33x2.70mm_HandSolder -> ZKU Capacitors:CAP_ZKU_F_PAN
- C4, C5: value 22uF -> 47uF; footprint Capacitor_SMD:C_1210_3225Metric_Pad1.33x2.70mm_HandSolder -> Capacitor_SMD:C_1206_3216Metric_Pad1.33x1.80mm_HandSolder
- C6: value 22uF X7R -> 4.7uF; footprint Capacitor_SMD:C_1210_3225Metric_Pad1.33x2.70mm_HandSolder -> Capacitor_SMD:C_0805_2012Metric_Pad1.18x1.45mm_HandSolder
- J1: value Conn_01x02 -> Conn_02x05_Odd_Even; footprint Connector_PinHeader_2.54mm:PinHeader_1x02_P2.54mm_Vertical -> Connector_PinHeader_2.54mm:PinHeader_2x05_P2.54mm_Vertical
- L1: footprint Inductor_SMD:L_Sumida_CDMC6D28_7.25x6.5mm -> Inductor:IND_SRP6530A_BRN
- R1, R2, R5: footprint Resistor_SMD:R_1210_3225Metric_Pad1.30x2.65mm_HandSolder -> Resistor_SMD:R_0805_2012Metric_Pad1.20x1.40mm_HandSolder
- R3: value 4.7k -> 49.9k; footprint Resistor_SMD:R_1210_3225Metric_Pad1.30x2.65mm_HandSolder -> Resistor_SMD:R_0805_2012Metric_Pad1.20x1.40mm_HandSolder
- moved C13 32.1 mm to (125.2, 64.4)
- moved C4 30.9 mm to (124.7, 84.6)
- moved C1 30.0 mm to (172.0, 77.6), turned to 180 degrees
- moved U1 27.5 mm to (175.9, 80.8)
- moved L1 27.1 mm to (175.6, 72.6)
- moved C2 25.1 mm to (179.7, 77.6), turned to 0 degrees
- moved J1 22.0 mm to (162.6, 76.9), turned to 0 degrees
- moved C6 20.5 mm to (145.8, 71.3)
- moved C11 20.5 mm to (134.5, 84.9)
- moved R3 17.8 mm to (141.0, 71.2)
- moved C5 17.6 mm to (124.7, 87.9), turned to 0 degrees
- moved R1 17.3 mm to (141.0, 65.3)
- moved C3 14.8 mm to (134.5, 80.7)
- moved C12 14.7 mm to (134.5, 89.2)
- moved R5 14.6 mm to (141.0, 77.1)
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Connections:
- C11 pad 2: GND -> GNDA
- C4 pad 1: +3.3V -> /VOUT
- C5 pad 1: Net-(U1-DITH_SYNC) -> /VOUT
- C6 pad 1: /VOUT -> +3.3V
- C6 pad 2: GND -> GNDA
- J1 pad 2: GND -> +12V
- R3 pad 2: GND -> GNDA
- R5 pad 2: Net-(C10-Pad1) -> GNDA
- U1 pad 13: /VOUT -> Net-(U1-ISN)
- U1 pad 14: GND -> unconnected-(U1-FB_INT_N-Pad14)
- U1 pad 16: Net-(U1-CDC) -> unconnected-(U1-CDC-Pad16)
- U1 pad 17: GND -> GNDA
- U1 pad 5: Net-(U1-DITH_SYNC) -> unconnected-(U1-DITH_SYNC-Pad5)
Routing:
- net GND: track 59.3 -> 0.00 mm
- net /VOUT: track 34.7 -> 0.00 mm
- net +3.3V: track 26.7 -> 0.00 mm, vias 2 -> 0
- net +12V: track 16.0 -> 0.00 mm
- net /EN: track 13.6 -> 0.00 mm, vias 1 -> 0
- net Net-(U1-COMP): track 8.04 -> 0.00 mm
- net Net-(U1-DITH_SYNC): track 8.01 -> 0.00 mm
- net Net-(U1-MODE): track 6.63 -> 0.00 mm
- net Net-(U1-EXTVCC): track 4.68 -> 0.00 mm
- net Net-(C10-Pad1): track 3.04 -> 0.00 mm
- net Net-(U1-BOOT2): track 5.51 -> 4.39 mm
- net Net-(U1-BOOT1): track 5.51 -> 4.52 mm
- added copper zone on In1.Cu, net GND
Other:
- board outline added: 25 x 25 mm
- copper layers 2 -> 4
