File: 12VBuckBoost.kicad_sch (KiCad schematic)
At the start: 24 parts, among them J1 Conn_01x02, J2 Conn_01x01, J3 QWIIC, J4 Conn_01x02, U1 TPS55289RYQR

Commit message: Init
Parts:
- removed C10: 22uF, Capacitor_SMD:C_1210_3225Metric_Pad1.33x2.70mm_HandSolder, symbol Device:C_Small
- removed C13, C7, C8, C9: 22uF X7R, Capacitor_SMD:C_1210_3225Metric_Pad1.33x2.70mm_HandSolder, symbol Device:C_Small
- removed J1, J4: Conn_01x02, Connector_PinHeader_2.54mm:PinHeader_1x02_P2.54mm_Vertical, symbol Connector_Generic:Conn_01x02
- removed J2: Conn_01x01, Connector_PinHeader_2.54mm:PinHeader_1x01_P2.54mm_Vertical, symbol Connector_Generic:Conn_01x01
- removed J3: QWIIC, Connector_JST:JST_PH_S4B-PH-K_1x04_P2.00mm_Horizontal, symbol Connector_Generic:Conn_01x04
- removed R6: 4.7k, Resistor_SMD:R_1210_3225Metric_Pad1.30x2.65mm_HandSolder, symbol Device:R_Small
- removed U1: TPS55289RYQR, TPS55289:RYQ0021A-MFG, symbol TPS55289:TPS55289RYQR
- added C13, C14: 330uF, ZKU Capacitors:CAP_ZKU_F_PAN, symbol Device:C_Polarized_Small
- added J1: Conn_02x05_Odd_Even, Connector_PinHeader_2.54mm:PinHeader_2x05_P2.54mm_Vertical, symbol Connector_Generic:Conn_02x05_Odd_Even
- added R4: 10m, Resistor_SMD:R_0805_2012Metric_Pad1.20x1.40mm_HandSolder, symbol Device:R_Small
- added U2: TPS55289RYQR, TPS55289:RYQ0021A-MFG, symbol TPS55289:TPS55289RYQR
- C1, C2: value 22uF -> 0.1uF; footprint Capacitor_SMD:C_1210_3225Metric_Pad1.33x2.70mm_HandSolder -> Capacitor_SMD:C_0805_2012Metric_Pad1.18x1.45mm_HandSolder
- C4, C5: value 22uF -> 47uF; footprint Capacitor_SMD:C_1210_3225Metric_Pad1.33x2.70mm_HandSolder -> Capacitor_SMD:C_1206_3216Metric_Pad1.33x1.80mm_HandSolder
- C6: value 22uF X7R -> 4.7uF; footprint Capacitor_SMD:C_1210_3225Metric_Pad1.33x2.70mm_HandSolder -> Capacitor_SMD:C_0805_2012Metric_Pad1.18x1.45mm_HandSolder
- L1: footprint Inductor_SMD:L_Sumida_CDMC6D28_7.25x6.5mm -> Inductor:IND_SRP6530A_BRN
- R1, R2, R5: footprint Resistor_SMD:R_1210_3225Metric_Pad1.30x2.65mm_HandSolder -> Resistor_SMD:R_0805_2012Metric_Pad1.20x1.40mm_HandSolder
- R3: value 4.7k -> 49.9k; footprint Resistor_SMD:R_1210_3225Metric_Pad1.30x2.65mm_HandSolder -> Resistor_SMD:R_0805_2012Metric_Pad1.20x1.40mm_HandSolder
Connections:
- net +12V: now also C13.1, J1.1 (Pin_1), J1.2 (Pin_2), U2.7 (VIN)
- net +3.3V: now also C6.1, J1.8 (Pin_8), U2.18 (VCC); no longer C4.1
- net EN: now also J1.10 (Pin_10), U2.1 (EN_UVLO)
- net GND: now also C13.2, C14.2, J1.5 (Pin_5), J1.6 (Pin_6), U2.9 (PGND); no longer C11.2, C6.2, R3.2
- net SCL: now also J1.7 (Pin_7), U2.3 (SCL)
- net SDA: now also J1.9 (Pin_9), U2.4 (SDA)
- net VOUT: now also C4.1, C5.1, C14.1, J1.3 (Pin_3), J1.4 (Pin_4), R4.2, U2.13 (ISN); no longer C6.1
- net at C11.1, R5.1: now also U2.15 (COMP)
- net GNDA: now reaches R5.2
- net GNDA: now also C11.2, C6.2, R3.2, U2.17 (AGND)
- net at C2.2: now also L1.1, U2.10 (SW2)
- net at R1.2: now also U2.2 (MODE)
- net at C1.2: now also L1.2, U2.8 (SW1)
- net at R2.2: now also U2.21 (EXTVCC)
- net at R3.1: now also U2.6 (FSW)
- net SW1: no longer names the net of C1.1
- net SW1: now also U2.20 (BOOT1); no longer L1.1
- net SW2: no longer names the net of C2.1
- net SW2: now also U2.19 (BOOT2); no longer L1.2
- new net: R4.1, U2.11 (VOUT), U2.12 (ISP)
- no-connect marks 0 -> 3
Other:
- moved on the sheet: C1, C11, C12, C2, C3, L1, R1, R2, R3, R5
